Commit message: 14050719

File: ros2_ws/src/my_robot/urdf/my_robot.urdf.xacro (robot description, xacro)
@@ -3,13 +3,28 @@
   <!-- ================= PARAMETERS ================= -->
   <xacro:property name="wheel_radius" value="0.06"/>         <!-- 6 cm -->
-  <xacro:property name="wheel_separation" value="0.50"/>     <!-- 50 cm -->
+  <!-- FIXED: was 0.50, but your measured value used everywhere else
+       (serial_odom_node.py, overview doc) is 0.48 m. Kept in sync now. -->
+  <xacro:property name="wheel_separation" value="0.48"/>     <!-- 48 cm, measured -->
   <xacro:property name="base_height" value="0.115"/>         <!-- 11.5 cm -->
   <xacro:property name="body_side" value="0.43"/>            <!-- 43 cm triangle sides -->
-  <xacro:property name="lidar_height" value="0.235"/>        <!-- 23.5 cm from ground -->
-  <xacro:property name="camera_height" value="0.20"/>        <!-- 20 cm from ground -->
+  <xacro:property name="caster_radius" value="0.03"/>
+  <xacro:property name="lidar_height" value="0.235"/>        <!-- 23.5 cm from GROUND -->
+  <xacro:property name="camera_height" value="0.20"/>        <!-- 20 cm from GROUND -->
   <xacro:property name="camera_tilt" value="-10"/>           <!-- downward 10 deg -->
-<!--  <xacro:property name="pi" value="3.141592653589793"/> -->      <!-- pi constant -->
+  <!-- 'pi' is a built-in xacro constant (math.pi) — no need to define it,
+       leaving it undefined does NOT break ${camera_tilt * pi / 180} below. -->
   <xacro:property name="mass_total" value="4.5"/>
   <xacro:property name="mass_wheel" value="0.25"/>
+  <!-- ================= MATERIALS (top-level, so they're globally valid) =========
+       FIXED: previously "gray" and "black" were only given a <color> the FIRST
+       time they appeared inside a link's <visual>, then reused bare
+       (<material name="gray"/>) in later links. That's not valid URDF — a
+       <material> only carries color info where it's declared, or if declared
+       once at the robot's top level. It happened to render in RViz because
+       RViz caches materials by name, but it's not guaranteed to work in
+       Gazebo or other tools. Declaring them once here fixes that for good. -->
+  <material name="white"><color rgba="1 1 1 1"/></material>
+  <material name="gray"><color rgba="0.3 0.3 0.3 1"/></material>
+  <material name="black"><color rgba="0 0 0 1"/></material>
   <!-- ================= BASE LINK ================= -->
   <link name="base_footprint" />
@@ -17,4 +32,7 @@
       <parent link="base_footprint"/>
       <child link="base_link"/>
+      <!-- base_link's origin sits one wheel-radius above the ground.
+           Everything below that is relative to THIS origin, not the ground -
+           this is the source of the old height bugs. -->
       <origin xyz="0 0 ${wheel_radius}" rpy="0 0 0" />
   </joint>
@@ -24,7 +42,5 @@
         <box size="${body_side} ${body_side} ${base_height}"/>
       </geometry>
-      <material name="white">
-        <color rgba="1 1 1 1"/>
-      </material>
+      <material name="white"/>
       <origin xyz="0 0 ${base_height/2}" rpy="0 0 0"/>
     </visual>
@@ -50,15 +66,11 @@
         <cylinder radius="${wheel_radius}" length="0.03"/>
       </geometry>
-      <material name="gray">
-        <color rgba="0.3 0.3 0.3 1"/>
-      </material>
-      <!-- FIXED: Origin should be at 0,0,0 since joint handles the transform -->
-      <origin xyz="0 0 0" rpy="1.5708 0 0"/>
-    </visual>
-    <collision>
-      <geometry>
-        <cylinder radius="${wheel_radius}" length="0.03"/>
-      </geometry>
-      <!-- FIXED: Origin should be at 0,0,0 since joint handles the transform -->
+      <material name="gray"/>
+      <origin xyz="0 0 0" rpy="1.5708 0 0"/>
+    </visual>
+    <collision>
+      <geometry>
+        <cylinder radius="${wheel_radius}" length="0.03"/>
+      </geometry>
       <origin xyz="0 0 0" rpy="1.5708 0 0"/>
     </collision>
@@ -74,5 +86,10 @@
     <parent link="base_link"/>
     <child link="left_wheel_link"/>
-    <origin xyz="0 ${wheel_separation/2} ${wheel_radius}" rpy="0 0 0"/>
+    <!-- FIXED: was z="${wheel_radius}", which DOUBLE-COUNTED the ground
+         clearance already applied by base_joint above. That put the wheel
+         centers 0.12 m up instead of 0.06 m, floating the wheels 6 cm off
+         the ground in the model. z=0 here is correct since base_link's
+         own origin is already at wheel-radius height. -->
+    <origin xyz="0 ${wheel_separation/2} 0" rpy="0 0 0"/>
     <axis xyz="0 1 0"/>
   </joint>
@@ -84,12 +101,10 @@
       </geometry>
       <material name="gray"/>
-      <!-- FIXED: Origin should be at 0,0,0 since joint handles the transform -->
-      <origin xyz="0 0 0" rpy="1.5708 0 0"/>
-    </visual>
-    <collision>
-      <geometry>
-        <cylinder radius="${wheel_radius}" length="0.03"/>
-      </geometry>
-      <!-- FIXED: Origin should be at 0,0,0 since joint handles the transform -->
+      <origin xyz="0 0 0" rpy="1.5708 0 0"/>
+    </visual>
+    <collision>
+      <geometry>
+        <cylinder radius="${wheel_radius}" length="0.03"/>
+      </geometry>
       <origin xyz="0 0 0" rpy="1.5708 0 0"/>
     </collision>
@@ -105,5 +120,6 @@
     <parent link="base_link"/>
     <child link="right_wheel_link"/>
-    <origin xyz="0 -${wheel_separation/2} ${wheel_radius}" rpy="0 0 0"/>
+    <!-- FIXED: same double-counted height bug as left wheel -->
+    <origin xyz="0 -${wheel_separation/2} 0" rpy="0 0 0"/>
     <axis xyz="0 1 0"/>
   </joint>
@@ -112,22 +128,28 @@
     <visual>
       <geometry>
-        <sphere radius="0.03"/>
-      </geometry>
-      <material name="gray"/>
-      <!-- FIXED: Origin should be at 0,0,0 since joint handles the transform -->
-      <origin xyz="0 0 0" rpy="0 0 0"/>
-    </visual>
-    <collision>
-      <geometry>
-        <sphere radius="0.03"/>
-      </geometry>
-      <!-- FIXED: Origin should be at 0,0,0 since joint handles the transform -->
-      <origin xyz="0 0 0" rpy="0 0 0"/>
-    </collision>
+        <sphere radius="${caster_radius}"/>
+      </geometry>
+      <material name="gray"/>
+      <origin xyz="0 0 0" rpy="0 0 0"/>
+    </visual>
+    <collision>
+      <geometry>
+        <sphere radius="${caster_radius}"/>
+      </geometry>
+      <origin xyz="0 0 0" rpy="0 0 0"/>
+    </collision>
+    <inertial>
+      <mass value="0.05"/>
+      <inertia ixx="0.00002" ixy="0" ixz="0" iyy="0.00002" iyz="0" izz="0.00002"/>
+    </inertial>
   </link>
   <joint name="rear_caster_joint" type="fixed">
     <parent link="base_link"/>
     <child link="rear_caster_link"/>
-    <origin xyz="-0.18 0 0.03" rpy="0 0 0"/>
+    <!-- FIXED: was z=0.03, which (combined with the wheel bug) floated the
+         caster ball 6 cm above the ground too. Ground is at z=-wheel_radius
+         relative to base_link, so to make the caster ball's SURFACE touch
+         the ground: z = -wheel_radius + caster_radius. -->
+    <origin xyz="-0.18 0 ${-wheel_radius + caster_radius}" rpy="0 0 0"/>
   </joint>
   <!-- ================= LIDAR ================= -->
@@ -137,14 +159,22 @@
         <cylinder radius="0.04" length="0.05"/>
       </geometry>
-      <material name="black">
-        <color rgba="0 0 0 1"/>
-      </material>
-      <origin xyz="0 0 0" rpy="0 0 0"/>
-    </visual>
+      <material name="black"/>
+      <origin xyz="0 0 0" rpy="0 0 0"/>
+    </visual>
+    <inertial>
+      <mass value="0.15"/>
+      <inertia ixx="0.00005" ixy="0" ixz="0" iyy="0.00005" iyz="0" izz="0.00005"/>
+    </inertial>
   </link>
   <joint name="lidar_joint" type="fixed">
     <parent link="base_link"/>
     <child link="lidar_link"/>
-    <origin xyz="0 0 ${lidar_height}" rpy="0 0 0"/>
+    <!-- FIXED: lidar_height (0.235 m) is documented as "from ground", but was
+         being applied directly as an offset from base_link, which itself is
+         already wheel_radius above ground. That put the real-world height at
+         wheel_radius + lidar_height = 0.295 m, not the intended 0.235 m.
+         Subtracting wheel_radius here makes the true ground height match
+         the property's comment/your measurement. -->
+    <origin xyz="0 0 ${lidar_height - wheel_radius}" rpy="0 0 0"/>
   </joint>
   <!-- ================= CAMERA ================= -->
@@ -157,9 +187,15 @@
       <origin xyz="0 0 0" rpy="0 0 0"/>
     </visual>
+    <inertial>
+      <mass value="0.05"/>
+      <inertia ixx="0.00002" ixy="0" ixz="0" iyy="0.00002" iyz="0" izz="0.00002"/>
+    </inertial>
   </link>
   <joint name="camera_joint" type="fixed">
     <parent link="base_link"/>
     <child link="camera_link"/>
-    <origin xyz="${body_side/2 - 0.02} 0 ${camera_height}" rpy="${camera_tilt * pi / 180} 0 0"/>
+    <!-- FIXED: same "from ground" vs "from base_link" mismatch as the lidar -->
+    <origin xyz="${body_side/2 - 0.02} 0 ${camera_height - wheel_radius}"
+            rpy="${camera_tilt * pi / 180} 0 0"/>
   </joint>
   <!-- ================= IMU ================= -->
@@ -172,11 +208,29 @@
       <origin xyz="0 0 0" rpy="0 0 0"/>
     </visual>
+    <inertial>
+      <mass value="0.02"/>
+      <inertia ixx="0.00001" ixy="0" ixz="0" iyy="0.00001" iyz="0" izz="0.00001"/>
+    </inertial>
   </link>
   <joint name="imu_joint" type="fixed">
     <parent link="base_link"/>
     <child link="imu_link"/>
+    <!-- Not documented as "from ground", so left as an offset from base_link
+         (sits just above the body's top face). Unchanged. -->
     <origin xyz="0 0 ${base_height + 0.01}" rpy="0 0 0"/>
   </joint>
-  <!-- ================= ROS2 CONTROL ================= -->
+  <!-- ================= ROS2 CONTROL =================
+       NOTE: this block is very likely dead weight right now. Your
+       robot.launch.py never starts controller_manager or spawns any
+       controllers — serial_odom_node.py talks to the Arduino directly and
+       owns /cmd_vel + /odom itself. Also, "diff_drive_controller/..." is a
+       *controller* plugin (belongs in a ros2_controllers.yaml loaded by
+       controller_manager), not a *hardware interface* plugin (what
+       <hardware><plugin> is supposed to reference — something implementing
+       hardware_interface::SystemInterface for your actual board). As written
+       this block won't do anything at runtime and would fail to load if you
+       ever did try to bring up controller_manager with it. Left in place
+       but flagged — remove it or replace it with a real hardware interface
+       plugin if you migrate to ros2_control later. -->
   <ros2_control name="TriangleBotSystem" type="system">
     <hardware>
